File: Electronic/Implementation/ZumoComSystem/IF_pololu.sch (KiCad schematic (older format))
At the start: 41 parts, among them J3 Left, J4 Conn_02x07_Odd_Even, J5 Right, J6 Conn_02x07_Odd_Even

Commit message: add charger
Connections:
- net Main_Switch: now also J3.16 (Pin_16); no longer J3.14 (Pin_14)
- net nBUTTON_A renamed BUT_A
- net nBUTTON_B: no longer names the net of Q?.2 (D), R?.2
- net nBUTTON_C: no longer names the net of Q?.2 (D), R?.2
- net nRemote_Butt_A: no longer names the net of Q?.1 (G), R?.1, R?.2
- net nRemote_Butt_B: no longer names the net of Q?.1 (G), R?.1, R?.2
- net nRemote_Butt_C: no longer names the net of Q?.1 (G), R?.1, R?.2
Other:
- moved on the sheet: R?, SW?
Changed lines of the file:
@@
 Wire Wire Line
 	9500 4400 9950 4400
-Text Label 2150 1200 0    50   ~ 0
+Text Label 2450 1200 2    50   ~ 0
 BUT_A
 $Comp
@@
 Text HLabel 1400 4600 0    50   Input ~ 0
 nLED_B
-Text HLabel 6950 1200 2    50   Output ~ 0
-nBUTTON_C
 $Comp
 L power:GND #PWR?
@@
 Wire Wire Line
 	2150 3300 2250 3300
-Text HLabel 4650 1200 2    50   Output ~ 0
-nBUTTON_B
-Text HLabel 2450 1200 2    50   Output ~ 0
-nBUTTON_A
 Wire Wire Line
 	2100 1750 2100 1950
-Text HLabel 1500 1550 0    50   Input ~ 0
-nRemote_Butt_A
 $Comp
 L power:+3.3V #PWR?
@@
 Wire Wire Line
 	2100 1200 2450 1200
-Wire Wire Line
-	1750 1450 1750 1550
 $Comp
 L power:GND #PWR?
@@
 Wire Wire Line
 	4300 1750 4300 1950
-Text HLabel 3700 1550 0    50   Input ~ 0
-nRemote_Butt_B
 $Comp
 L power:+3.3V #PWR?
@@
 $EndComp
 Wire Wire Line
-	4300 1200 4650 1200
-Wire Wire Line
 	3950 1450 3950 1550
 $Comp
 L Switch:SW_Push SW?
 U 1 1 61349AA0
-P 3550 2000
-F 0 "SW?" V 3504 2148 50  0000 L CNN
-F 1 "SW_Push" V 3595 2148 50  0000 L CNN
-F 2 "" H 3550 2200 50  0001 C CNN
-F 3 "~" H 3550 2200 50  0001 C CNN
-	1    3550 2000
+P 3550 1750
+F 0 "SW?" V 3504 1898 50  0000 L CNN
+F 1 "SW_Push" V 3595 1898 50  0000 L CNN
+F 2 "" H 3550 1950 50  0001 C CNN
+F 3 "~" H 3550 1950 50  0001 C CNN
+	1    3550 1750
 	0    -1   -1   0
 $EndComp
@@
 L power:GND #PWR?
 U 1 1 61349AA8
-P 3550 2200
-F 0 "#PWR?" H 3550 1950 50  0001 C CNN
-F 1 "GND" H 3555 2027 50  0000 C CNN
-F 2 "" H 3550 2200 50  0001 C CNN
-F 3 "" H 3550 2200 50  0001 C CNN
-	1    3550 2200
+P 3550 1950
+F 0 "#PWR?" H 3550 1700 50  0001 C CNN
+F 1 "GND" H 3555 1777 50  0000 C CNN
+F 2 "" H 3550 1950 50  0001 C CNN
+F 3 "" H 3550 1950 50  0001 C CNN
+	1    3550 1950
 	1    0    0    -1
 $EndComp
@@
 Wire Wire Line
 	6600 1750 6600 1950
-Text HLabel 6000 1550 0    50   Input ~ 0
-nRemote_Butt_C
 $Comp
 L power:+3.3V #PWR?
@@
 	1    0    0    -1
 $EndComp
-Wire Wire Line
-	6600 1350 6600 1200
-Wire Wire Line
-	6600 1200 6950 1200
 Wire Wire Line
 	6250 1450 6250 1550
@@
 Text Label 2750 4150 0    50   ~ 0
 LED_B*
-Text GLabel 5450 4600 1    50   Input ~ 0
+Text GLabel 6000 4400 1    50   Input ~ 0
 VBAT_ZCS
 Wire Wire Line
-	5450 4600 5450 4700
-Wire Wire Line
-	5450 4700 5200 4700
+	6000 4400 6000 4700
+Wire Wire Line
+	6000 4700 5200 4700
 NoConn ~ 4700 3500
 NoConn ~ 5200 3500
@@
 NoConn ~ 5200 3900
 NoConn ~ 5200 4000
-NoConn ~ 5200 4200
+NoConn ~ 5200 4100
 NoConn ~ 5200 4300
 NoConn ~ 5200 4400
@@
 L Device:R R?
 U 1 1 617380EC
-P 3800 1800
-F 0 "R?" V 3593 1800 50  0000 C CNN
-F 1 "R" V 3684 1800 50  0000 C CNN
-F 2 "" V 3730 1800 50  0001 C CNN
-F 3 "~" H 3800 1800 50  0001 C CNN
-	1    3800 1800
+P 3750 1550
+F 0 "R?" V 3543 1550 50  0000 C CNN
+F 1 "R" V 3634 1550 50  0000 C CNN
+F 2 "" V 3680 1550 50  0001 C CNN
+F 3 "~" H 3750 1550 50  0001 C CNN
+	1    3750 1550
 	0    1    1    0
 $EndComp
 Wire Wire Line
-	3550 1800 3650 1800
-Wire Wire Line
-	3950 1550 3950 1800
+	3550 1550 3600 1550
+Wire Wire Line
+	3950 1550 3900 1550
 Connection ~ 6250 1550
 Wire Wire Line
 	6250 1550 6300 1550
-Wire Wire Line
-	6000 1550 6250 1550
 Connection ~ 3950 1550
 Wire Wire Line
 	3950 1550 4000 1550
-Wire Wire Line
-	3700 1550 3950 1550
 $Comp
 L Switch:SW_Push SW?
 U 1 1 617BFBA9
-P 5850 2000
-F 0 "SW?" V 5804 2148 50  0000 L CNN
-F 1 "SW_Push" V 5895 2148 50  0000 L CNN
-F 2 "" H 5850 2200 50  0001 C CNN
-F 3 "~" H 5850 2200 50  0001 C CNN
-	1    5850 2000
+P 5850 1750
+F 0 "SW?" V 5804 1898 50  0000 L CNN
+F 1 "SW_Push" V 5895 1898 50  0000 L CNN
+F 2 "" H 5850 1950 50  0001 C CNN
+F 3 "~" H 5850 1950 50  0001 C CNN
+	1    5850 1750
 	0    -1   -1   0
 $EndComp
@@
 L power:GND #PWR?
 U 1 1 617BFBAF
-P 5850 2200
-F 0 "#PWR?" H 5850 1950 50  0001 C CNN
-F 1 "GND" H 5855 2027 50  0000 C CNN
-F 2 "" H 5850 2200 50  0001 C CNN
-F 3 "" H 5850 2200 50  0001 C CNN
-	1    5850 2200
+P 5850 1950
+F 0 "#PWR?" H 5850 1700 50  0001 C CNN
+F 1 "GND" H 5855 1777 50  0000 C CNN
+F 2 "" H 5850 1950 50  0001 C CNN
+F 3 "" H 5850 1950 50  0001 C CNN
+	1    5850 1950
 	1    0    0    -1
 $EndComp
@@
 L Device:R R?
 U 1 1 617BFBB5
-P 6100 1800
-F 0 "R?" V 5893 1800 50  0000 C CNN
-F 1 "R" V 5984 1800 50  0000 C CNN
-F 2 "" V 6030 1800 50  0001 C CNN
-F 3 "~" H 6100 1800 50  0001 C CNN
-	1    6100 1800
+P 6050 1550
+F 0 "R?" V 5843 1550 50  0000 C CNN
+F 1 "R" V 5934 1550 50  0000 C CNN
+F 2 "" V 5980 1550 50  0001 C CNN
+F 3 "~" H 6050 1550 50  0001 C CNN
+	1    6050 1550
 	0    1    1    0
 $EndComp
 Wire Wire Line
-	5850 1800 5950 1800
-Wire Wire Line
-	6250 1550 6250 1800
-Connection ~ 1750 1550
-Wire Wire Line
-	1750 1550 1800 1550
-Wire Wire Line
-	1500 1550 1750 1550
+	5850 1550 5900 1550
+Wire Wire Line
+	6250 1550 6200 1550
+Wire Wire Line
+	1700 1550 1750 1550
 $Comp
 L Switch:SW_Push SW?
 U 1 1 617DBB37
-P 1350 2000
-F 0 "SW?" V 1304 2148 50  0000 L CNN
-F 1 "SW_Push" V 1395 2148 50  0000 L CNN
-F 2 "" H 1350 2200 50  0001 C CNN
-F 3 "~" H 1350 2200 50  0001 C CNN
-	1    1350 2000
+P 1350 1750
+F 0 "SW?" V 1304 1898 50  0000 L CNN
+F 1 "SW_Push" V 1395 1898 50  0000 L CNN
+F 2 "" H 1350 1950 50  0001 C CNN
+F 3 "~" H 1350 1950 50  0001 C CNN
+	1    1350 1750
 	0    -1   -1   0
 $EndComp
@@
 L power:GND #PWR?
 U 1 1 617DBB3D
-P 1350 2200
-F 0 "#PWR?" H 1350 1950 50  0001 C CNN
-F 1 "GND" H 1355 2027 50  0000 C CNN
-F 2 "" H 1350 2200 50  0001 C CNN
-F 3 "" H 1350 2200 50  0001 C CNN
-	1    1350 2200
+P 1350 1950
+F 0 "#PWR?" H 1350 1700 50  0001 C CNN
+F 1 "GND" H 1355 1777 50  0000 C CNN
+F 2 "" H 1350 1950 50  0001 C CNN
+F 3 "" H 1350 1950 50  0001 C CNN
+	1    1350 1950
 	1    0    0    -1
 $EndComp
@@
 L Device:R R?
 U 1 1 617DBB43
-P 1600 1800
-F 0 "R?" V 1393 1800 50  0000 C CNN
-F 1 "R" V 1484 1800 50  0000 C CNN
-F 2 "" V 1530 1800 50  0001 C CNN
-F 3 "~" H 1600 1800 50  0001 C CNN
-	1    1600 1800
+P 1550 1550
+F 0 "R?" V 1343 1550 50  0000 C CNN
+F 1 "R" V 1434 1550 50  0000 C CNN
+F 2 "" V 1480 1550 50  0001 C CNN
+F 3 "~" H 1550 1550 50  0001 C CNN
+	1    1550 1550
 	0    1    1    0
 $EndComp
 Wire Wire Line
-	1350 1800 1450 1800
-Wire Wire Line
-	1750 1550 1750 1800
+	1350 1550 1400 1550
 $Comp
 L power:GND #PWR?
@@
 Text HLabel 5050 6250 0    50   Input ~ 0
 nON_OFF
-Text Label 5750 4100 2    50   ~ 0
+Text Label 5750 4200 2    50   ~ 0
 Main_Switch
 Wire Wire Line
-	5750 4100 5200 4100
+	5750 4200 5200 4200
 $Comp
 L power:+3.3V #PWR?
@@
 	1    0    0    -1
 $EndComp
-Wire Wire Line
-	4300 1350 4300 1200
 $Comp
 L power:+3.3V #PWR?
@@
 Wire Wire Line
 	2100 1200 2100 1100
-Connection ~ 4300 1200
-Wire Wire Line
-	4300 1200 4300 1100
-Connection ~ 6600 1200
-Wire Wire Line
-	6600 1200 6600 1100
 Wire Wire Line
 	7900 5200 7900 5550
@@
 	7900 4550 7900 4700
 Connection ~ 7900 4700
+Wire Wire Line
+	4300 1100 4300 1350
+Wire Wire Line
+	6600 1100 6600 1350
+Wire Wire Line
+	1750 1450 1750 1550
+Connection ~ 1750 1550
+Wire Wire Line
+	1750 1550 1800 1550
 $EndSCHEMATC

Commit message: Electronic: no charger, added Cp2102 instead of Ft232, first palcement
Parts:
- removed Q? (x8): Q_NMOS_GDS, symbol Device:Q_NMOS_GDS
- added Q10, Q11, Q12, Q5, Q6, Q7, Q8, Q9: AO3414, Package_TO_SOT_SMD:SOT-23, symbol Device:Q_NMOS_GSD
- D10: renamed from D?; value LED -> LED, green; footprint (none) -> LED_SMD:LED_0603_1608Metric_Pad1.05x0.95mm_HandSolder
- D11: renamed from D?; value LED -> LED, blue; footprint (none) -> LED_SMD:LED_0603_1608Metric_Pad1.05x0.95mm_HandSolder
- D9: renamed from D?; value LED -> LED, red; footprint (none) -> LED_SMD:LED_0603_1608Metric_Pad1.05x0.95mm_HandSolder
- J3, J5: footprint Connector_PinHeader_2.54mm:PinHeader_2x13_P2.54mm_Vertical_SMD -> footprints:PinHeader_2x13_SMD_bottom
- J6: footprint Connector_PinSocket_2.54mm:PinSocket_2x07_P2.54mm_Vertical_SMD -> footprints:PinSocket_2x07_P2.54mm_Vertical_SMD
- R24, R36, R41: renamed from R?; value R -> 0; footprint (none) -> Resistor_SMD:R_0603_1608Metric_Pad1.05x0.95mm_HandSolder
- R25, R32, R37, R38, R39, R40, R42, R43, R44, R45: renamed from R?; footprint (none) -> Resistor_SMD:R_0603_1608Metric_Pad1.05x0.95mm_HandSolder
- R26, R28, R33: renamed from R?; value R -> 300; footprint (none) -> Resistor_SMD:R_0603_1608Metric_Pad1.05x0.95mm_HandSolder
- R27, R29, R31: renamed from R?; value R -> 10k; footprint (none) -> Resistor_SMD:R_0603_1608Metric_Pad1.05x0.95mm_HandSolder
- R30: renamed from R?; value R -> 180; footprint (none) -> Resistor_SMD:R_0603_1608Metric_Pad1.05x0.95mm_HandSolder
- R34, R35: renamed from R?; value R -> 150; footprint (none) -> Resistor_SMD:R_0603_1608Metric_Pad1.05x0.95mm_HandSolder
- SW3, SW4, SW5: renamed from SW?; footprint (none) -> Button_Switch_SMD:SW_SPST_B3U-1000P-B
- gave numbers to parts that had none: 1
Connections:
- net VBAT_ZCS is gone; now on net +5V: J3.26 (Pin_26)
- net +3V3: no longer D12.4 (A)
- net +5V: now also D12.4 (A)
- net GND: now also Q10.2 (S), Q11.2 (S), Q12.2 (S), Q5.2 (S), Q6.2 (S), Q7.2 (S), Q8.2 (S), Q9.2 (S)
- net Main_Switch: now also Q10.3 (D)
- net nLED_A: now also Q6.1 (G)
- net nLED_B: now also Q7.1 (G)
- net nLED_C: now also Q8.1 (G)
- net nON_OFF: now also Q10.1 (G)
- net nRESET: now also Q12.3 (D)
- net nRST: now also Q12.1 (G)
- net at R24.1, R25.2: now also Q5.1 (G)
- net at R36.1, R37.2: now also Q9.1 (G)
- net at R38.2: now also Q9.3 (D)
- net at R41.1, R42.2: now also Q11.1 (G)
- net nBUT_C: now reaches R43.2
- net nBUT_C: now also Q11.3 (D)
- net BUT_A renamed nBUT_A
- net nBUT_A: now also Q5.3 (D)
- net LED_A* renamed LED_A
- net LED_A: now also Q6.3 (D)
- net LED_B* renamed LED_B
- net LED_B: now also Q7.3 (D)
- net LED_C* renamed LED_C
- net LED_C: now also Q8.3 (D)
Other:
- note added: "Batteriespannung Zumo"
- moved on the sheet: D11, R30, R31

Commit message: Electronic: PCB routed
Parts:
- renumbered Q8 to Q10, Q9 to Q11, Q10 to Q12, Q11 to Q13, Q12 to Q14, Q5 to Q7, Q6 to Q8, Q7 to Q9, R24 to R21, R25 to R22, R26 to R23, R27 to R24, R28 to R25, R29 to R26, R30 to R27, R31 to R28, R32 to R29, R33 to R30, R34 to R31, R35 to R32, R36 to R33, R37 to R34, R38 to R35, R39 to R36, R40 to R37, R41 to R38, R42 to R39, R43 to R40, R44 to R41, R45 to R42
Connections:
- net nBUT_B: now also Q11.3 (D), R35.2
Other:
- note added: "I_max = 2.6 A"

Commit message: Electronic: implementation of the connector for external charging (reverse polarity protected)
Parts:
- renumbered D12 to D10, D9 to D7, D10 to D8, D11 to D9, J3 to J4, J4 to J5, J5 to J6, J6 to J7, Q11 to Q10, Q12 to Q11, Q13 to Q12, Q14 to Q13, Q7 to Q6, Q8 to Q7, Q9 to Q8, Q10 to Q9, R21 to R16, R22 to R17, R23 to R18, R24 to R19, R25 to R20, R26 to R21, R27 to R22, R28 to R23, R29 to R24, R30 to R25, R31 to R26, R32 to R27, R33 to R28, R34 to R29, R35 to R30, R36 to R31, R37 to R32, R38 to R33, R39 to R34, R40 to R35, R41 to R36, R42 to R37
Other:
- note added: "Battery Voltage Zumo"
- note removed: "Batteriespannung Zumo"
