File: Electronic/Implementation/ZumoComSystem/ZumoComSystem.sch (KiCad schematic (older format))
At the start: 0 parts

Commit message: Coutouts, BOM, ...
Changed lines of the file:
@@
 Sheet 1 7
 Title "Zumo Communication System"
-Date "2022-03-25"
+Date "2022-04-15"
 Rev "V1.0"
 Comp "NewTec GmbH"
@@
 F5 "MISO" O L 6500 4900 50
 F6 "MOSI" B L 6500 4800 50
+F7 "ESP_EN" B L 6500 5300 50
 $EndSheet
 $Sheet
@@
 F18 "nBUT_C" I R 8000 1650 50
 F19 "nBUT_A" I R 8000 1450 50
+F20 "ESP_EN" B L 6500 2400 50
 $EndSheet
 Wire Wire Line
@@
 Wire Wire Line
 	5500 2100 6500 2100
+Wire Wire Line
+	6500 2400 5700 2400
+Wire Wire Line
+	5700 2400 5700 5300
+Wire Wire Line
+	5700 5300 6500 5300
 $EndSCHEMATC

Commit message: After Review: - optimized 3V3 and 5V regulator - Vias placement - optimized routing - add Newtec Logo (again) - add Repository Name
Parts:
- added L1: NewTec_Logo, footprints:NT_Kicad_Logo_2500x2500, symbol NewTec_Logo:NewTec_Logo
Changed lines of the file:
@@
 Sheet 1 7
 Title "Zumo Communication System"
-Date "2022-08-05"
+Date "2022-08-11"
 Rev "V1.1"
 Comp "NewTec GmbH"
@@
 EndData
 $EndBitmap
+$Comp
+L NewTec_Logo:NewTec_Logo L1
+U 1 1 62F4D7EF
+P 750 7700
+F 0 "L1" H 750 7800 50  0001 C CNN
+F 1 "NewTec_Logo" H 750 7700 50  0000 C CNN
+F 2 "footprints:NT_Kicad_Logo_2500x2500" H 750 7700 50  0001 C CNN
+F 3 "" H 750 7700 50  0001 C CNN
+	1    750  7700
+	1    0    0    -1
+$EndComp
 $EndSCHEMATC
