File: Electronic/Implementation/ZumoComSystem/power_reg.sch (KiCad schematic (older format))
At the start: 15 parts, among them Q1 PMOS_GSD-TSM260P02CX RFG, SW1 MLL1200S, U1 LT1374CS8-5PBF, U2 ADP2370ACPZ-3.3-R7

Commit message: #93 ESP32 3V3 Diode; U_Bat_Meas from Pin IO2 to IO13; Test-Vias D+,D-
Parts:
- renumbered R3 to R1
Changed lines of the file:
@@
 	7400 1500 7850 1500
 $Comp
-L Device:R R3
+L Device:R R1
 U 1 1 6262337C
 P 6200 850
-F 0 "R3" V 5993 850 50  0000 C CNN
+F 0 "R1" V 5993 850 50  0000 C CNN
 F 1 "10k" V 6084 850 50  0000 C CNN
 F 2 "Resistor_SMD:R_0603_1608Metric_Pad1.05x0.95mm_HandSolder" V 6130 850 50  0001 C CNN
@@
 	4450 3700 8650 3700
 $Comp
-L power:+5V #PWR?
+L power:+5V #PWR02
 U 1 1 62EA39DD
 P 3600 3500
-F 0 "#PWR?" H 3600 3350 50  0001 C CNN
+F 0 "#PWR02" H 3600 3350 50  0001 C CNN
 F 1 "+5V" H 3615 3673 50  0000 C CNN
 F 2 "" H 3600 3500 50  0001 C CNN

Commit message: select the right footprint for the Diode (D7)
Parts:
- D2: footprint Diode_SMD:D_SOD-323 -> Diode_SMD:D_SOD-323_HandSoldering
Changed lines of the file:
@@
 F 0 "D2" H 8900 3917 50  0000 C CNN
 F 1 "30V 100mA" H 8900 3826 50  0000 C CNN
-F 2 "Diode_SMD:D_SOD-323" H 8900 3700 50  0001 C CNN
+F 2 "Diode_SMD:D_SOD-323_HandSoldering" H 8900 3700 50  0001 C CNN
 F 3 "https://www.comchiptech.com/admin/files/product/SS8050-G%20RevA181526.pdf" H 8900 3700 50  0001 C CNN
 F 4 "SMC Diode Solutions" H 8900 3700 50  0001 C CNN "Manufacturer"

Commit message: update Date, footprints, ...
Parts:
- L2: footprint Inductor_SMD:L_Vishay_IHLP-4040 -> footprints:L_Vishay_IHLP-4040_3D
Changed lines of the file:
@@
 Sheet 2 7
 Title "Zumo Communication System"
-Date "2022-05-27"
+Date "2022-08-04"
 Rev "V1.1"
 Comp "NewTec GmbH"
@@
 F 0 "L2" V 9140 4200 50  0000 C CNN
 F 1 "15u" V 9049 4200 50  0000 C CNN
-F 2 "Inductor_SMD:L_Vishay_IHLP-4040" H 8950 4200 50  0001 C CNN
+F 2 "footprints:L_Vishay_IHLP-4040_3D" H 8950 4200 50  0001 C CNN
 F 3 "https://www.mouser.de/datasheet/2/427/lp40dz5a-1762293.pdf" H 8950 4200 50  0001 C CNN
 F 4 " Vishay / Dale " H 8950 4200 50  0001 C CNN "Manufacturer"

Commit message: After Review: - optimized 3V3 and 5V regulator - Vias placement - optimized routing - add Newtec Logo (again) - add Repository Name
Parts:
- renumbered L1 to L2, L2 to L3
Changed lines of the file:
@@
 Sheet 2 7
 Title "Zumo Communication System"
-Date "2022-08-05"
+Date "2022-08-11"
 Rev "V1.1"
 Comp "NewTec GmbH"
@@
 $EndComp
 $Comp
-L Device:L L2
+L Device:L L3
 U 1 1 60C6A253
 P 8950 4200
-F 0 "L2" V 9140 4200 50  0000 C CNN
+F 0 "L3" V 9140 4200 50  0000 C CNN
 F 1 "15u" V 9049 4200 50  0000 C CNN
 F 2 "footprints:L_Vishay_IHLP-4040_3D" H 8950 4200 50  0001 C CNN
@@
 $EndComp
 $Comp
-L Device:L L1
+L Device:L L2
 U 1 1 60C698F7
 P 8000 1500
-F 0 "L1" V 8190 1500 50  0000 C CNN
+F 0 "L2" V 8190 1500 50  0000 C CNN
 F 1 "6.8u" V 8099 1500 50  0000 C CNN
 F 2 "footprints:L_Coilcraft_XxL4040_Handsolder" H 8000 1500 50  0001 C CNN

Commit message: #95 START Hardware-Version v1.2 - L2: pad size increased - some small fixes
Parts:
- renumbered L2 to L1, L3 to L2
Connections:
- net at C1.1, C2.1, Q1.3 (D)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: no longer C3.1, U1.6 (VC)
- new net: C3.1, U1.6 (VC)
Changed lines of the file:
@@
 Sheet 2 7
 Title "Zumo Communication System"
-Date "2022-08-11"
-Rev "V1.1"
+Date "2022-09-05"
+Rev "V1.2"
 Comp "NewTec GmbH"
 Comment1 "Schneider, Niklas"
@@
 Wire Wire Line
 	3950 2000 3950 3450
-Connection ~ 8050 4400
 Connection ~ 3950 3450
 Wire Wire Line
@@
 $EndComp
 $Comp
-L Device:L L3
+L Device:L L2
 U 1 1 60C6A253
 P 8950 4200
-F 0 "L3" V 9140 4200 50  0000 C CNN
+F 0 "L2" V 9140 4200 50  0000 C CNN
 F 1 "15u" V 9049 4200 50  0000 C CNN
 F 2 "footprints:L_Vishay_IHLP-4040_3D" H 8950 4200 50  0001 C CNN
@@
 $EndComp
 $Comp
-L Device:L L2
+L Device:L L1
 U 1 1 60C698F7
 P 8000 1500
-F 0 "L2" V 8190 1500 50  0000 C CNN
+F 0 "L1" V 8190 1500 50  0000 C CNN
 F 1 "6.8u" V 8099 1500 50  0000 C CNN
 F 2 "footprints:L_Coilcraft_XxL4040_Handsolder" H 8000 1500 50  0001 C CNN
@@
 Wire Wire Line
 	7850 4300 8050 4300
-Connection ~ 8050 4300
-Wire Wire Line
-	8050 4300 8050 4400
 Connection ~ 8650 3700
 Wire Wire Line
