File: Electronic/Implementation/ZumoComSystem/Battery.kicad_sch (KiCad schematic)
At the start: 29 parts, among them IC1 S-8252AAL-M6T1U, IC2 MCP73844-840I_MS, J6 PJ-090BH, Q2 RQ5E065AJTCL, Q3 RQ5E065AJTCL, Q4 Q_PMOS_GSD, SW5 SW_Push

Commit message: HW: Version 2.0 Layout, BOM, Gerber-files created
Parts:
- D10: footprint Diode_SMD:D_SMB_Handsoldering -> footprints:D_SMB_Handsoldering
Changed lines of the file:
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@@
   (title_block
     (title "ZumoComSystem")
-    (date "2023-12-05")
+    (date "2023-12-18")
     (rev "2.0")
     (company "NewTec GmbH")
@@
       (effects (font (size 1.27 1.27)) (justify left))
     )
-    (property "Footprint" "Diode_SMD:D_SMB_Handsoldering" (at 238.76 78.74 0)
-      (effects (font (size 1.27 1.27)) hide)
-    )
+    (property "Footprint" "footprints:D_SMB_Handsoldering" (at 238.76 78.74 0)
+      (effects (font (size 1.27 1.27)) hide)
+    )
